File: rpi_absorbance.kicad_pcb (KiCad board)
At the start: 2 copper layers, 39.2 x 56.1 mm, 33 parts, among them CON1 BARREL_JACK, P1 CONN_02X04, P2 CONN_01X02, P3 RPI_HEADER, P4 STEPPER_CONN, P5 CONN_02X06, Q1 ZTX692B, U1 R-78B5.0-1.5L, U2 NXP_PUMH10, U3 DRV8825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

Commit message: Update resistors
Parts:
- R1, R7, R8: footprint Resistors_SMD:R_0805_HandSoldering -> Resistors_SMD:R_0603_HandSoldering
- moved R8 0.25 mm to (173.5, 95.8)
Routing:
- net +5V: track 97.7 -> 90.3 mm
- net /5vSCL: track 5.72 -> 6.25 mm

Commit message: Update pcb
Parts:
- moved D1 0.41 mm to (152.8, 127.7)
Routing:
- net GND: track 84.7 -> 103.1 mm, vias 39 -> 45
